File: FOC_CONTROLLER_V2/FOC_CONTROLLER_V2.kicad_pcb (KiCad board)
At the start: 4 copper layers, 80 x 80 mm, 120 parts, among them IC1 STSPIN32G4, J10 AZ1117, J11 T1M-04-GF-DH, J12 Conn_01x06, J2 Conn_01x01, J4 Conn_01x01, Q1 CSD18543Q3A, Q2 CSD19534Q5A, Q3 CSD19534Q5A, Q4 CSD18543Q3A, Q5 CSD19534Q5A, Q6 CSD18543Q3A, U1 THVD1400

Commit message: PCB DRIVER : Graphics
Parts:
- added G***: LOGO, LOGO, F.Cu at (171.7, 124.7)
- added TP1: 3V3, TestPoint:TestPoint_Pad_D1.0mm, F.Cu at (132.7, 114.7)
- added TP14: 5V, TestPoint:TestPoint_Pad_D1.0mm, F.Cu at (165.9, 98.2)
- added TP15: 5V, TestPoint:TestPoint_Pad_D1.0mm, F.Cu at (158.8, 98.2)
- added TP2: 3V3, TestPoint:TestPoint_Pad_D1.0mm, F.Cu at (134.8, 112.7)
- added TP3: 3V3, TestPoint:TestPoint_Pad_D1.0mm, F.Cu at (132.1, 111.5)
- added TP4: 3V3, TestPoint:TestPoint_Pad_D1.0mm, F.Cu at (128.9, 112.4)
- C16: renamed from 1  2
- D1: renamed from LED 1
- D3: renamed from LED 2
- J1: renamed from DC IN
- R6: renamed from GATE HIGH
- renumbered BOOT to C1, 5V to D8, 3v3 to D9, RS485 to H1, V to J3, JTAG to J6, Encoder to R44, Adress to SW3, USER to User1
Routing:
- net /PB7: track 0.00 -> 29.5 mm, vias 0 -> 2
- net /PB6: track 0.00 -> 26.0 mm, vias 0 -> 2
- net +3.3V: track 77.5 -> 61.1 mm
- net Net-(IC1-PD2): track 64.6 -> 73.0 mm
- net Net-(IC1-PB4): track 60.3 -> 67.5 mm
- net /UART_TX: track 23.6 -> 21.7 mm
- net /UART_RX: track 15.8 -> 14.7 mm
- net /VCP_RX: track 82.2 -> 83.2 mm
- net Net-(IC1-PB5): track 72.6 -> 73.5 mm
- net GND: vias 340 -> 349
Other:
- board text added: "3V3"
- board text added: "3V3EXT"
- board text added: "5V"
- board text added: "ADRESS"
- board text added: "BOOT"
- board text added: "DC IN"
- board text added: "ENCODER"
- board text added: "GATE HIGH"
- board text added: "JTAG"
- board text added: "LED 1"
- board text added: "LED 2"
- board text added: "LSW1"
- board text added: "LSW2"
- board text added: "NTC"
- board text added: "PB6"
- board text added: "PB7"
- board text added: "RS485"
- board text added: "U V W"
- board text removed: "Motion System"
- board text removed: "TDI"
- board text removed: "U"
- board text removed: "W"

Commit message: Communication board : done
Parts:
- moved C30 9.76 mm to (122.1, 121.9), turned to -90 degrees
- moved PwrJumper1 4.26 mm to (129.1, 123.0)
- renumbered User1 to User
Routing:
- net Net-(PwrJumper1-C): track 13.2 -> 0.00 mm
- net +3.3V: track 61.1 -> 55.9 mm
- net +3,3V_EXT: track 7.45 -> 6.16 mm
- net /VCP_TX: track 77.0 -> 76.2 mm
- net /VCP_RX: track 83.2 -> 83.9 mm
- net GND: vias 349 -> 353
- added copper zone on F.Cu, net Net-(PwrJumper1-C)
Other:
- board text added: "FOC Motor Driver v2.0 Design by Bilal YOUSFI"
- board text removed: "FOC Motor Driver v2.0 Designed by Bilal YOUSFI"
